File: Clock_M-D.sch (EAGLE design)
At the start: 60 parts, among them IC1 ATMEGA328P, IC2 LM4040....., IC3 REG1117, IC4 MCP6002_, J1 THONKICONNNEW, J2 THONKICONNNEW, J20 ICSP, J3 THONKICONNNEW, J4 THONKICONNNEW, J5 THONKICONNNEW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

Commit message: Add files via upload
Parts:
- IC2: value LM4040..... -> LM40405.0
Changed lines of the file:
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@@
 <part name="R8" library="rcl" library_urn="urn:adsk.eagle:library:334" deviceset="R-US_" device="R0805" package3d_urn="urn:adsk.eagle:package:23553/2" value="1K"/>
 <part name="FRAME1" library="frames" library_urn="urn:adsk.eagle:library:229" deviceset="FRAME_A_L" device=""/>
-<part name="IC2" library="texas" library_urn="urn:adsk.eagle:library:387" deviceset="LM4041" device="DBZ" package3d_urn="urn:adsk.eagle:package:7566925/3" technology="A12" value="LM4040....."/>
+<part name="IC2" library="texas" library_urn="urn:adsk.eagle:library:387" deviceset="LM4041" device="DBZ" package3d_urn="urn:adsk.eagle:package:7566925/3" technology="A12" value="LM40405.0"/>
 <part name="SUPPLY2" library="supply2" library_urn="urn:adsk.eagle:library:372" deviceset="GND" device=""/>
 <part name="SUPPLY3" library="supply2" library_urn="urn:adsk.eagle:library:372" deviceset="GND" device=""/>
